File: PCBFiles/Snowduino Null.kicad_sch (KiCad schematic)
At the start: 86 parts

Commit message: Add files via upload
Parts:
- removed C? (x8): 0.1uF, Capacitor_SMD:C_0603_1608Metric, symbol Device:C_Small
- removed C? (x2): 10uF, Capacitor_SMD:C_0805_2012Metric, symbol Device:C_Small
- removed C? (x2): 47pF, Capacitor_SMD:C_0603_1608Metric, symbol Device:C_Small
- removed C?: 100pF, Capacitor_SMD:C_0603_1608Metric, symbol Device:C_Small
- removed C? (x2): 22pF, Capacitor_SMD:C_0603_1608Metric, symbol Device:C_Small
- removed C?: 10n, Capacitor_SMD:C_0603_1608Metric, symbol Device:C
- removed C?: 47u, Capacitor_SMD:CP_Elec_6.3x3.9, symbol Device:C_Small
- removed C?: 100n, Capacitor_SMD:C_0603_1608Metric, symbol Device:C_Small
- removed C?: 4.7nF, Capacitor_SMD:C_0603_1608Metric, symbol Device:C
- removed C?: 0.01uF, Capacitor_SMD:C_0603_1608Metric, symbol Device:C_Small
- removed C? (x2): 47u, Capacitor_SMD:CP_Elec_6.3x3.9, symbol Device:C
- removed C?: 1uF, Capacitor_SMD:C_0805_2012Metric, symbol Device:C_Small
- removed C?: 4u7, Capacitor_SMD:C_0603_1608Metric, symbol Device:C_Small
- removed C?: 4.7uF, Capacitor_SMD:C_0805_2012Metric, symbol Uno-rescue:CP1_Small-Device
- removed D? (x5): WHITE, LED_SMD:LED_0603_1608Metric, symbol Uno-rescue:LED_ALT-Device
- removed D? (x3): D_Schottky, Diode_SMD:D_SOD-123F, symbol Device:D_Schottky
- removed F?: MF-MSMF050-2, Fuse:Fuse_1812_4532Metric, symbol Device:Polyfuse
- removed FB? (x2): 470r, Resistor_SMD:R_0603_1608Metric, symbol Uno-rescue:Ferrite_Bead_Small-Device
- removed FID? (x2): Fiducial, Fiducial:Fiducial_0.75mm_Mask1.5mm, symbol Mechanical:Fiducial
- removed H? (x4): MountingHole, MountingHole:MountingHole_3.2mm_M3, symbol Mechanical:MountingHole
- removed J?: USB_C_Receptacle_USB2.0, Connector_USB:USB_C_Receptacle_HRO_TYPE-C-31-M-12, symbol Connector:USB_C_Receptacle_USB2.0
- removed J?: JTAG, Connector_PinHeader_1.27mm:PinHeader_2x05_P1.27mm_Vertical, symbol Connector:Conn_ARM_JTAG_SWD_10
- removed J?: ANALOG, Connector_PinSocket_2.54mm:PinSocket_1x06_P2.54mm_Vertical, symbol Connector_Generic:Conn_01x06
- removed J?: ICSP, Connector_PinHeader_2.54mm:PinHeader_2x03_P2.54mm_Vertical, symbol Connector_Generic:Conn_02x03_Odd_Even
- removed J?: POWER, Connector_PinSocket_2.54mm:PinSocket_1x08_P2.54mm_Vertical, symbol Connector_Generic:Conn_01x08
- removed J?: DIGITAL-HIGH, Connector_PinSocket_2.54mm:PinSocket_1x10_P2.54mm_Vertical, symbol Connector_Generic:Conn_01x10
- removed J?: Conn_01x04, Connector_PinHeader_2.54mm:PinHeader_1x04_P2.54mm_Vertical, symbol Connector_Generic:Conn_01x04
- removed J?: DIGITAL-LOW, Connector_PinSocket_2.54mm:PinSocket_1x08_P2.54mm_Vertical, symbol Connector_Generic:Conn_01x08
- removed J?: PJ-202A, KiCad2:DC005G25A20, symbol Connector:Barrel_Jack_Switch
- removed JP?: RESET-EN, Jumper:SolderJumper-2_P1.3mm_Bridged_RoundedPad1.0x1.5mm, symbol Jumper:Jumper_2_Bridged
- removed L?: 10u, Inductor_SMD:L_6.3x6.3_H3, symbol Device:L
- removed Q? (x2): 2N7002E, Package_TO_SOT_SMD:SOT-23, symbol Transistor_FET:2N7002E
- removed Q?: 2N7002, Package_TO_SOT_SMD:SOT-23, symbol Transistor_FET:2N7002
- removed Q?: Q_NMOS_DGS, Package_TO_SOT_SMD:TSOT-23, symbol Device:Q_NMOS_DGS
- removed R? (x5): 330, Resistor_SMD:R_0603_1608Metric, symbol Device:R
- removed R? (x2): 52K3, Resistor_SMD:R_0603_1608Metric, symbol Device:R_US
- removed R? (x5): 10k, Resistor_SMD:R_0603_1608Metric, symbol Device:R_US
- removed R?: 1M, Resistor_SMD:R_0603_1608Metric, symbol Device:R
- removed R? (x2): 5.1k, Resistor_SMD:R_0603_1608Metric, symbol Device:R
- removed R?: 330r, Resistor_SMD:R_0603_1608Metric, symbol Device:R_US
- removed R? (x2): 52K3, Resistor_SMD:R_0603_1608Metric, symbol Device:R
- removed R?: 52k3, Resistor_SMD:R_0603_1608Metric, symbol Device:R
- removed R?: 1k, Resistor_SMD:R_0603_1608Metric, symbol Device:R_US
- removed R? (x2): 27r, Resistor_SMD:R_0603_1608Metric, symbol Device:R_US
- removed SW?: SW_SPST, KiCad:PTS641SM31SMTR2LFS, symbol Switch:SW_SPST
- removed U?: AP1117-33, Package_TO_SOT_SMD:SOT-223-3_TabPin2, symbol Regulator_Linear:AP1117-33
- removed U?: ATSAMC21G, Package_QFP:TQFP-48_7x7mm_P0.5mm, symbol FortyTwoLabs:ATSAMC21G
- removed U?: FT231XQ, Package_DFN_QFN:QFN-20-1EP_4x4mm_P0.5mm_EP2.5x2.5mm, symbol Interface_USB:FT231XQ
- removed U?: USBLC6-2SC6, Package_TO_SOT_SMD:SOT-23-6, symbol Power_Protection:USBLC6-2SC6
- removed U?: LM2734Y, Package_TO_SOT_SMD:TSOT-23-6, symbol Regulator_Switching:LM2734Y
- removed Y?: 32.768kHz, Crystal:Crystal_SMD_MicroCrystal_CC7V-T1A-2Pin_3.2x1.5mm, symbol Device:Crystal_Small
- added C1, C2: 22pF, Capacitor_SMD:C_0603_1608Metric, symbol Device:C_Small
- added C10, C15, C18, C22, C6, C7, C8, C9: 0.1uF, Capacitor_SMD:C_0603_1608Metric, symbol Device:C_Small
- added C11: 4.7nF, Capacitor_SMD:C_0603_1608Metric, symbol Device:C
- added C12, C4: 10uF, Capacitor_SMD:C_0805_2012Metric, symbol Device:C_Small
- added C13: 10nF, Capacitor_SMD:C_0603_1608Metric, symbol Device:C_Small
- added C14: 4.7uF, Capacitor_SMD:C_0805_2012Metric, symbol Uno-rescue:CP1_Small-Device
- added C16, C17: 47pF, Capacitor_SMD:C_0603_1608Metric, symbol Device:C_Small
- added C19: 100n, Capacitor_SMD:C_0603_1608Metric, symbol Device:C_Small
- added C20, C24: 47u, Capacitor_SMD:CP_Elec_6.3x3.9, symbol Device:C
- added C21: 4u7, Capacitor_SMD:C_0603_1608Metric, symbol Device:C_Small
- added C23: 10n, Capacitor_SMD:C_0603_1608Metric, symbol Device:C
- added C26: 47u, Capacitor_SMD:CP_Elec_6.3x3.9, symbol Device:C_Small
- added C3: 100pF, Capacitor_SMD:C_0603_1608Metric, symbol Device:C_Small
- added C5: 1uF, Capacitor_SMD:C_0805_2012Metric, symbol Device:C_Small
- added D1, D2, D3, D4, D5: WHITE, LED_SMD:LED_0603_1608Metric, symbol Uno-rescue:LED_ALT-Device
- added D6, D7, D8: D_Schottky, Diode_SMD:D_SOD-123F, symbol Device:D_Schottky
- added D9: D_Schottky, Diode_SMD:D_SOD-323, symbol Device:D_Schottky
- added F1: MF-MSMF050-2, Fuse:Fuse_1812_4532Metric, symbol Device:Polyfuse
- added FB1, FB2: 470r, Resistor_SMD:R_0603_1608Metric, symbol Uno-rescue:Ferrite_Bead_Small-Device
- added H1, H2, H3, H4: MountingHole, MountingHole:MountingHole_3.2mm_M3, symbol Mechanical:MountingHole
- added J1: JTAG, Connector_PinHeader_1.27mm:PinHeader_2x05_P1.27mm_Vertical, symbol Connector:Conn_ARM_JTAG_SWD_10
- added J2: POWER, Connector_PinSocket_2.54mm:PinSocket_1x08_P2.54mm_Vertical, symbol Connector_Generic:Conn_01x08
- added J3: ANALOG, Connector_PinSocket_2.54mm:PinSocket_1x06_P2.54mm_Vertical, symbol Connector_Generic:Conn_01x06
- added J4: ICSP, Connector_PinHeader_2.54mm:PinHeader_2x03_P2.54mm_Vertical, symbol Connector_Generic:Conn_02x03_Odd_Even
- added J5: USB_C_Receptacle_USB2.0, Connector_USB:USB_C_Receptacle_HRO_TYPE-C-31-M-12, symbol Connector:USB_C_Receptacle_USB2.0
- added J6: DIGITAL-HIGH, Connector_PinSocket_2.54mm:PinSocket_1x10_P2.54mm_Vertical, symbol Connector_Generic:Conn_01x10
- added J7: DIGITAL-LOW, Connector_PinSocket_2.54mm:PinSocket_1x08_P2.54mm_Vertical, symbol Connector_Generic:Conn_01x08
- added J8: Conn_01x04, Connector_PinHeader_2.54mm:PinHeader_1x04_P2.54mm_Vertical, symbol Connector_Generic:Conn_01x04
- added J9: PJ-202A, KiCad2:DC005G25A20, symbol Connector:Barrel_Jack_Switch
- added JP1: RESET-EN, Jumper:SolderJumper-2_P1.3mm_Bridged_RoundedPad1.0x1.5mm, symbol Jumper:Jumper_2_Bridged
- added JP2: RESET-EN, Connector_PinHeader_1.27mm:PinHeader_1x02_P1.27mm_Vertical, symbol Jumper:Jumper_2_Bridged
- added L1: 10u, Inductor_SMD:L_6.3x6.3_H3, symbol Device:L
- added Q1, Q2: 2N7002E, Package_TO_SOT_SMD:SOT-23, symbol Transistor_FET:2N7002E
- added Q3, Q5: Q_PMOS_GSD, Package_TO_SOT_SMD:SOT-23, symbol Device:Q_PMOS_GSD
- added Q4: 2N7002, Package_TO_SOT_SMD:SOT-23, symbol Transistor_FET:2N7002
- added R1: 330r, Resistor_SMD:R_0603_1608Metric, symbol Device:R_US
- added R10, R11: 27r, Resistor_SMD:R_0603_1608Metric, symbol Device:R_US
- added R12, R13, R14, R17, R9: 330, Resistor_SMD:R_0603_1608Metric, symbol Device:R
- added R15, R16: 52K3, Resistor_SMD:R_0603_1608Metric, symbol Device:R_US
- added R18: 52k3, Resistor_SMD:R_0603_1608Metric, symbol Device:R
- added R19, R2, R20, R4, R5: 10k, Resistor_SMD:R_0603_1608Metric, symbol Device:R_US
- added R21, R22: 52K3, Resistor_SMD:R_0603_1608Metric, symbol Device:R
- added R23, R6: 1M, Resistor_SMD:R_0603_1608Metric, symbol Device:R
- added R3: 1k, Resistor_SMD:R_0603_1608Metric, symbol Device:R_US
- added R7, R8: 5.1k, Resistor_SMD:R_0603_1608Metric, symbol Device:R
- added SW1: SW_Push_Dual, KiCad:PTS641SM31SMTR2LFS, symbol Switch:SW_Push_Dual
- added U1: ATSAMC21G, Package_QFP:TQFP-48_7x7mm_P0.5mm, symbol FortyTwoLabs:ATSAMC21G
- added U2: USBLC6-2SC6, Package_TO_SOT_SMD:SOT-23-6, symbol Power_Protection:USBLC6-2SC6
- added U3: FT231XQ, Package_DFN_QFN:QFN-20-1EP_4x4mm_P0.5mm_EP2.5x2.5mm, symbol Interface_USB:FT231XQ
- added U4: LM2734Y, Package_TO_SOT_SMD:TSOT-23-6, symbol Regulator_Switching:LM2734Y
- added U5: AP1117-33, Package_TO_SOT_SMD:SOT-223-3_TabPin2, symbol Regulator_Linear:AP1117-33
- added Y1: 32.768kHz, Crystal:Crystal_SMD_MicroCrystal_CC7V-T1A-2Pin_3.2x1.5mm, symbol Device:Crystal_Small
Connections:
- net +12V: now also C20.2, D6.1 (K), J2.8 (Pin_8), R15.1, R18.1, U4.5 (VIN)
- net +3V3: now also C26.1, D9.2 (A), J2.4 (Pin_4), R12.1, R13.1, R9.1, U5.2 (VO)
- net +5V: now also C24.1, D7.2 (A), J2.5 (Pin_5), J4.2 (Pin_2), JP2.2 (B), L1.2, Q3.2 (S), Q5.2 (S), R21.1, U5.3 (VI)
- net A0-DAC: now also J3.1 (Pin_1), U1.3 (PA02)
- net A1: now also J3.2 (Pin_2), U1.7 (PB08)
- net A2: now also J3.3 (Pin_3), U1.8 (PB09)
- net A3: now also J3.4 (Pin_4), U1.9 (PA04)
- net A4: now also J3.5 (Pin_5), U1.10 (PA05)
- net A5: now also J3.6 (Pin_6), U1.47 (PB02)
- net AREF: now also C19.1, C21.1, J6.8 (Pin_8), U1.4 (PA03)
- net CAN0-RX: now also J8.3 (Pin_3), U1.34 (PA25)
- net CAN0-TX: now also J8.2 (Pin_2), U1.33 (PA24)
- net CON-D+: now also J5.A6 (D+), J5.B6 (D+), U2.4 (I/O2)
- net CON-D-: now also J5.A7 (D-), J5.B7 (D-), U2.6 (I/O1)
- net D0: now also J7.1 (Pin_1), U1.16 (PA11)
- net D1: now also J7.2 (Pin_2), U1.15 (PA10)
- net D10: now also J6.3 (Pin_3), U1.27 (PA18)
- net D11: now also J6.4 (Pin_4), U1.25 (PA16)
- net D12: now also J6.5 (Pin_5), U1.28 (PA19)
- net D13: now also J6.6 (Pin_6), Q2.1 (G), U1.26 (PA17)
- net D2: now also J7.3 (Pin_3), U1.23 (PA14)
- net D3: now also J7.4 (Pin_4), U1.14 (PA09)
- net D4: now also J7.5 (Pin_5), U1.13 (PA08)
- net D5: now also J7.6 (Pin_6), U1.24 (PA15)
- net D6: now also J7.7 (Pin_7), U1.29 (PA20)
- net D7: now also J7.8 (Pin_8), U1.30 (PA21)
- net D8: now also J6.1 (Pin_1), U1.11 (PA06)
- net D9: now also J6.2 (Pin_2), U1.12 (PA07)
- net ESD-D+: now also C16.1, R11.2, U2.3 (I/O2)
- net ESD-D-: now also C17.1, R10.2, U2.1 (I/O1)
- net FTDI-3.3V: now also C18.1, Q4.1 (G), R14.1, R17.1, R19.1, U3.10 (3V3OUT), U3.11 (~{RESET}), U3.20 (VCCIO)
- net FTDI-D+: now also R11.1, U3.8 (USBDP)
- net FTDI-D-: now also R10.1, U3.9 (USBDM)
- net GND: now also C1.2, C10.2, C11.1, C12.2, C13.2, C14.2, C15.2, C16.2, C17.2, C18.2, C19.2, C2.2, C20.1, C21.2, C24.2, C26.2, C4.2, C5.2, C6.2, C7.2, C8.2, C9.2, D2.1 (K), D8.2 (A), J1.3 (GND), J1.5 (GND), J2.6 (Pin_6), J2.7 (Pin_7), J4.6 (Pin_6), J5.A1 (GND), J5.A12 (GND), J5.B1 (GND), J5.B12 (GND), J6.7 (Pin_7), J8.1 (Pin_1), J9.2, J9.3, Q1.2 (S), Q2.2 (S), R16.2, R22.2, R23.1, R6.2, R7.2, R8.1, SW1.1, SW1.3, U1.18 (GND), U1.35 (GND), U1.42 (GND), U1.5 (GNDANA), U2.2 (GND), U3.13 (GND), U3.21 (GND), U3.3 (GND), U4.2 (GND), U5.1 (GND)
- net LED-RX: now also D4.1 (K), U3.14 (CBUS1)
- net LED-TX: now also D5.1 (K), U3.7 (CBUS2)
- net MISO: now also J4.1 (Pin_1), U1.21 (PA12)
- net MOSI-CAN1-TX: now also J4.4 (Pin_4), U1.19 (PB10)
- net PA13: now also U1.22 (PA13)
- net PA27: now also U1.39 (PA27)
- net PA28: now also U1.41 (PA28)
- net PB03: now also U1.48 (PB03)
- net SAM-~{RESET}: now also C3.2, J1.10 (~{RESET}), J2.3 (Pin_3), J4.5 (Pin_5), JP1.2 (B), R1.1, R2.1, U1.40 (~{RESET})
- net SCK-CAN1-RX: now also J4.3 (Pin_3), U1.20 (PB11)
- net SCL: now also J6.10 (Pin_10), R5.1, U1.32 (PA23)
- net SDA: now also J6.9 (Pin_9), R4.1, U1.31 (PA22)
- net SWCLK: now also J1.4 (SWDCLK/TCK), R3.2, U1.45 (PA30)
- net SWDIO: now also J1.2 (SWDIO/TMS), Q1.1 (G), U1.46 (PA31)
- net UART-IN: now also U1.37 (PB22), U3.1 (RXD)
- net UART-OUT: now also U1.38 (PB23), U3.17 (TXD)
- net VBUS: now also C14.1, C15.1, F1.1, Q3.3 (D), U2.5 (VBUS), U3.12 (VCC)
- net ~{DTR}: now also Q4.2 (S), R19.2, U3.18 (~{DTR})
- new net: C1.1, U1.1 (PA00), Y1.1
- new net: C2.1, U1.2 (PA01), Y1.2
- new net: C5.1, C7.1, U1.43 (VDDCORE)
- new net: C10.1, C12.1, FB1.2, U1.6 (VDDANA)
- new net: D1.1 (K), Q2.3 (D)
- new net: D1.2 (A), R12.2
- new net: R1.2, SW1.2, SW1.4
- new net: D2.2 (A), R13.2
- new net: C23.2, D8.1 (K), L1.1, U4.6 (SW)
- new net: C13.1, FB2.2, J5.A4 (VBUS), J5.A9 (VBUS), J5.B4 (VBUS), J5.B9 (VBUS)
- new net: J5.A5 (CC1), R7.1
- new net: J5.B5 (CC2), R8.2
- new net: C11.2, J5.S1 (SHIELD), R6.1
- new net: JP2.1 (A), Q5.1 (G), R23.2
- new net: C22.2, Q4.3 (D), R20.2
- new net: C22.1, JP1.1 (A)
- new net: C23.1, D7.1 (K), U4.1 (BOOST)
- new net: R21.2, R22.1, U4.3 (FB)
- new net: D6.2 (A), J9.1
- new net: D3.1 (K), Q1.3 (D)
- new net: D3.2 (A), R9.2
- new net: F1.2, FB2.1
- new net: R18.2, U4.4 (EN)
- new net: Q3.1 (G), R15.2, R16.1
- new net: D4.2 (A), R14.2
- new net: D5.2 (A), R17.2
- new net +4V: C3.1, C4.1, C6.1, C8.1, C9.1, D9.1 (K), FB1.1, J1.1 (VTref), J2.2 (Pin_2), J8.4 (Pin_4), Q5.3 (D), R2.2, R20.1, R3.1, R4.2, R5.2, U1.17 (VDDIO), U1.36 (VDDIO), U1.44 (VDDIN)
Other:
- company: Snowduino.cc -> FortyTwo Systems
- title: Snowduino Null -> Uno

Commit message: Add files via upload
Parts:
- removed C20, C24: 47u, Capacitor_SMD:CP_Elec_6.3x3.9, symbol Device:C
- removed C26: 47u, Capacitor_SMD:CP_Elec_6.3x3.9, symbol Device:C_Small
- added C20, C24, C26: 47uF, Capacitor_SMD:CP_Elec_6.3x3.9, symbol Device:C_Polarized_US
Connections:
- net +12V: now also C20.1
- net +3V3: now also C26.1
- net +5V: now also C24.1
- net GND: now also C20.2, C24.2, C26.2
Changed lines of the file:
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@@
   (junction (at 27.94 168.91) (diameter 0) (color 0 0 0 0)
   )
+  (junction (at 370.84 166.37) (diameter 0) (color 0 0 0 0)
+  )
   (junction (at 208.28 191.77) (diameter 0.9144) (color 0 0 0 0)
   )
@@
   (junction (at 289.56 99.06) (diameter 0) (color 0 0 0 0)
   )
+  (junction (at 370.84 59.69) (diameter 0) (color 0 0 0 0)
+  )
   (junction (at 318.77 219.71) (diameter 0.9144) (color 0 0 0 0)
   )
@@
   (junction (at 208.28 207.01) (diameter 0.9144) (color 0 0 0 0)
   )
-  (junction (at 370.84 166.37) (diameter 0) (color 0 0 0 0)
-  )
   (junction (at 161.29 222.25) (diameter 0.9144) (color 0 0 0 0)
   )
@@
   (junction (at 17.78 168.91) (diameter 0) (color 0 0 0 0)
   )
-  (junction (at 370.84 59.69) (diameter 0) (color 0 0 0 0)
-  )
   (junction (at 88.9 77.47) (diameter 0.9144) (color 0 0 0 0)
   )
@@
     (pin "1")
   )
+  (symbol (lib_id "Device:C_Polarized_US") (at 370.84 170.18 0) (unit 1)
+    (in_bom yes) (on_board yes) (fields_autoplaced)
+    (property "Reference" "C26" (id 0) (at 374.015 168.2749 0)
+      (effects (font (size 1.27 1.27)) (justify left))
+    )
+    (property "Value" "47uF" (id 1) (at 374.015 170.8149 0)
+      (effects (font (size 1.27 1.27)) (justify left))
+    )
+    (property "Footprint" "Capacitor_SMD:CP_Elec_6.3x3.9" (id 2) (at 370.84 170.18 0)
+      (effects (font (size 1.27 1.27)) hide)
+    )
+    (property "Datasheet" "~" (id 3) (at 370.84 170.18 0)
+      (effects (font (size 1.27 1.27)) hide)
+    )
+    (pin "1")
+    (pin "2")
+  )
   (symbol (lib_id "Transistor_FET:2N7002") (at 311.15 217.17 270) (unit 1)
     (in_bom yes) (on_board yes)
@@
     (pin "2")
   )
+  (symbol (lib_id "Device:C_Polarized_US") (at 302.26 53.34 180) (unit 1)
+    (in_bom yes) (on_board yes) (fields_autoplaced)
+    (property "Reference" "C20" (id 0) (at 306.07 52.7049 0)
+      (effects (font (size 1.27 1.27)) (justify right))
+    )
+    (property "Value" "47uF" (id 1) (at 306.07 55.2449 0)
+      (effects (font (size 1.27 1.27)) (justify right))
+    )
+    (property "Footprint" "Capacitor_SMD:CP_Elec_6.3x3.9" (id 2) (at 302.26 53.34 0)
+      (effects (font (size 1.27 1.27)) hide)
+    )
+    (property "Datasheet" "~" (id 3) (at 302.26 53.34 0)
+      (effects (font (size 1.27 1.27)) hide)
+    )
+    (pin "1")
+    (pin "2")
+  )
   (symbol (lib_id "Device:C") (at 344.17 55.88 0) (unit 1)
     (in_bom yes) (on_board yes) (fields_autoplaced)
@@
     (pin "1")
   )
-  (symbol (lib_id "Device:C") (at 374.65 59.69 90) (unit 1)
-    (in_bom yes) (on_board yes) (fields_autoplaced)
-    (property "Reference" "C24" (id 0) (at 374.65 52.07 90))
-    (property "Value" "47u" (id 1) (at 374.65 54.61 90))
-    (property "Footprint" "Capacitor_SMD:CP_Elec_6.3x3.9" (id 2) (at 378.46 58.7248 0)
-      (effects (font (size 1.27 1.27)) hide)
-    )
-    (property "Datasheet" "~" (id 3) (at 374.65 59.69 0)
-      (effects (font (size 1.27 1.27)) hide)
-    )
-    (pin "1")
-    (pin "2")
-  )
   (symbol (lib_id "Device:R") (at 366.395 99.695 0) (unit 1)
     (in_bom yes) (on_board yes) (fields_autoplaced)
@@
     (pin "2")
   )
-  (symbol (lib_id "Device:C_Small") (at 370.84 168.91 0) (unit 1)
-    (in_bom yes) (on_board yes)
-    (property "Reference" "C26" (id 0) (at 373.1768 167.7416 0)
-      (effects (font (size 1.27 1.27)) (justify left))
-    )
-    (property "Value" "47u" (id 1) (at 373.1768 170.053 0)
-      (effects (font (size 1.27 1.27)) (justify left))
-    )
-    (property "Footprint" "Capacitor_SMD:CP_Elec_6.3x3.9" (id 2) (at 370.84 168.91 0)
-      (effects (font (size 1.27 1.27)) hide)
-    )
-    (property "Datasheet" "~" (id 3) (at 370.84 168.91 0)
-      (effects (font (size 1.27 1.27)) hide)
-    )
-    (pin "1")
-    (pin "2")
-  )
   (symbol (lib_id "Device:R") (at 351.79 67.31 0) (unit 1)
     (in_bom yes) (on_board yes) (fields_autoplaced)
@@
       (effects (font (size 1.27 1.27)) hide)
     )
-    (property "Value" "+3.3V" (id 1) (at 371.221 161.9758 0))
+    (property "Value" "+3.3V" (id 1) (at 373.38 158.75 0))
     (property "Footprint" "" (id 2) (at 370.84 166.37 0)
       (effects (font (size 1.27 1.27)) hide)
@@
     (pin "1")
   )
+  (symbol (lib_id "Device:C_Polarized_US") (at 374.65 59.69 90) (unit 1)
+    (in_bom yes) (on_board yes) (fields_autoplaced)
+    (property "Reference" "C24" (id 0) (at 374.015 52.07 90))
+    (property "Value" "47uF" (id 1) (at 374.015 54.61 90))
+    (property "Footprint" "Capacitor_SMD:CP_Elec_6.3x3.9" (id 2) (at 374.65 59.69 0)
+      (effects (font (size 1.27 1.27)) hide)
+    )
+    (property "Datasheet" "~" (id 3) (at 374.65 59.69 0)
+      (effects (font (size 1.27 1.27)) hide)
+    )
+    (pin "1")
+    (pin "2")
+  )
   (symbol (lib_id "power:+3.3V") (at 370.967 87.63 90) (unit 1)
     (in_bom yes) (on_board yes)
@@
     (pin "1")
   )
-  (symbol (lib_id "power:GND") (at 370.84 171.45 0) (unit 1)
+  (symbol (lib_id "power:GND") (at 370.84 173.99 0) (unit 1)
     (in_bom yes) (on_board yes)
-    (property "Reference" "#PWR064" (id 0) (at 370.84 177.8 0)
+    (property "Reference" "#PWR064" (id 0) (at 370.84 180.34 0)
       (effects (font (size 1.27 1.27)) hide)
     )
-    (property "Value" "GND" (id 1) (at 370.967 175.8442 0))
-    (property "Footprint" "" (id 2) (at 370.84 171.45 0)
+    (property "Value" "GND" (id 1) (at 370.967 178.3842 0))
+    (property "Footprint" "" (id 2) (at 370.84 173.99 0)
       (effects (font (size 1.27 1.27)) hide)
     )
-    (property "Datasheet" "" (id 3) (at 370.84 171.45 0)
+    (property "Datasheet" "" (id 3) (at 370.84 173.99 0)
       (effects (font (size 1.27 1.27)) hide)
     )
@@
     (pin "2")
   )
-  (symbol (lib_id "Device:C") (at 302.26 53.34 0) (unit 1)
-    (in_bom yes) (on_board yes) (fields_autoplaced)
-    (property "Reference" "C20" (id 0) (at 306.07 52.0699 0)
-      (effects (font (size 1.27 1.27)) (justify left))
-    )
-    (property "Value" "47u" (id 1) (at 306.07 54.6099 0)
-      (effects (font (size 1.27 1.27)) (justify left))
-    )
-    (property "Footprint" "Capacitor_SMD:CP_Elec_6.3x3.9" (id 2) (at 303.2252 57.15 0)
-      (effects (font (size 1.27 1.27)) hide)
-    )
-    (property "Datasheet" "~" (id 3) (at 302.26 53.34 0)
-      (effects (font (size 1.27 1.27)) hide)
-    )
-    (pin "1")
-    (pin "2")
-  )
   (symbol (lib_id "power:GND") (at 92.71 201.93 90) (unit 1)
     (in_bom yes) (on_board yes) (fields_autoplaced)
@@
       (reference "C19") (unit 1) (value "100n") (footprint "Capacitor_SMD:C_0603_1608Metric")
     )
-    (path "/f70b5175-705d-4781-8d75-54ebd03ff66e"
-      (reference "C20") (unit 1) (value "47u") (footprint "Capacitor_SMD:CP_Elec_6.3x3.9")
+    (path "/1f62e8f1-428b-4c31-b894-6c15cfae70f2"
+      (reference "C20") (unit 1) (value "47uF") (footprint "Capacitor_SMD:CP_Elec_6.3x3.9")
     )
     (path "/29102478-099d-49cb-8df9-b1efbe8c6adf"
@@
       (reference "C23") (unit 1) (value "10n") (footprint "Capacitor_SMD:C_0603_1608Metric")
     )
-    (path "/31693bcb-e71c-4eae-ac61-1ee67b70608e"
-      (reference "C24") (unit 1) (value "47u") (footprint "Capacitor_SMD:CP_Elec_6.3x3.9")
+    (path "/abca0a47-2387-453f-95e3-ceb75edca22c"
+      (reference "C24") (unit 1) (value "47uF") (footprint "Capacitor_SMD:CP_Elec_6.3x3.9")
     )
-    (path "/3f44e56b-06fb-4a81-96f5-e3128ffe9d91"
-      (reference "C26") (unit 1) (value "47u") (footprint "Capacitor_SMD:CP_Elec_6.3x3.9")
+    (path "/0fccc3c1-5c9d-4f5b-9ee8-b94233903abf"
+      (reference "C26") (unit 1) (value "47uF") (footprint "Capacitor_SMD:CP_Elec_6.3x3.9")
     )
     (path "/00000000-0000-0000-0000-00005f96fc5e"

Commit message: Add files via upload
Parts:
- R22: value 52K3 -> 10K
Changed lines of the file:
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@@
       (effects (font (size 1.27 1.27)) (justify left))
     )
-    (property "Value" "52K3" (id 1) (at 354.33 76.1999 0)
+    (property "Value" "10K" (id 1) (at 354.33 76.1999 0)
       (effects (font (size 1.27 1.27)) (justify left))
     )
@@
     )
     (path "/aa5a9908-1af2-474c-827c-a5f2274b4d23"
-      (reference "R22") (unit 1) (value "52K3") (footprint "Resistor_SMD:R_0603_1608Metric")
+      (reference "R22") (unit 1) (value "10K") (footprint "Resistor_SMD:R_0603_1608Metric")
     )
     (path "/31722a14-7c0c-48ed-a9ba-b6a2e0a2f3ad"
