File: PCBFiles/Snowduino Null.kicad_pcb (KiCad board)
At the start: 2 copper layers, 68.5 x 53.3 mm, 90 parts, among them J1 JTAG, J2 POWER, J3 ANALOG, J4 ICSP, J5 USB_C_Receptacle_USB2.0, J6 DIGITAL-HIGH, J7 DIGITAL-LOW, J8 Conn_01x04, J9 PJ-202A, Q1 2N7002E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

Commit message: Add files via upload
Parts:
- moved G*** 1.89 mm to (100.9, 102.8)

Commit message: Add files via upload
Parts:
- added D9: D_Schottky, Diode_SMD:D_SOD-323, F.Cu at (127.1, 105.6)
- added JP2: RESET-EN, Connector_PinHeader_1.27mm:PinHeader_1x02_P1.27mm_Vertical, F.Cu at (143.2, 87.7)
- added Q5: Q_PMOS_GSD, Package_TO_SOT_SMD:SOT-23, F.Cu at (119.4, 96.1)
- added R23: 1M, Resistor_SMD:R_0603_1608Metric, F.Cu at (116.1, 97.2)
- Q3: value Q_NMOS_DGS -> Q_PMOS_GSD; footprint Package_TO_SOT_SMD:TSOT-23 -> Package_TO_SOT_SMD:SOT-23
- SW1: value SW_SPST -> SW_Push_Dual
- moved G*** 1.71 mm to (100.4, 101.2)
Connections:
- C3 pad 1: +5V -> +4V
- C4 pad 1: +5V -> +4V
- C6 pad 1: +5V -> +4V
- C8 pad 1: +5V -> +4V
- C9 pad 1: +5V -> +4V
- FB1 pad 1: +5V -> +4V
- J1 pad 1: +5V -> +4V
- J2 pad 2: +5V -> +4V
- J8 pad 4: +3V3 -> +4V
- Q3 pad 1: +5V -> Net-(R15-Pad2)
- Q3 pad 2: Net-(Q3-Pad2) -> +5V
- R15 pad 2: Net-(Q3-Pad2) -> Net-(R15-Pad2)
- R16 pad 1: Net-(Q3-Pad2) -> Net-(R15-Pad2)
- R2 pad 2: +5V -> +4V
- R20 pad 1: +5V -> +4V
- R3 pad 1: +5V -> +4V
- R4 pad 2: +5V -> +4V
- R5 pad 2: +5V -> +4V
- U1 pad 17: +5V -> +4V
- U1 pad 36: +5V -> +4V
- U1 pad 44: +5V -> +4V
Routing:
- net +4V: track 0.00 -> 132.5 mm, vias 0 -> 10
- net Net-(JP2-Pad1): track 0.00 -> 38.1 mm, vias 0 -> 3
- net +5V: track 123.6 -> 88.4 mm, vias 9 -> 5
- net +3V3: track 61.5 -> 48.8 mm, vias 4 -> 2
- net GND: track 148.3 -> 160.4 mm, vias 89 -> 138
- net Net-(R15-Pad2): track 0.00 -> 4.97 mm
- net Net-(Q3-Pad2): track 3.67 -> 0.00 mm
- net /FTDI-3.3V: track 24.6 -> 26.1 mm, vias 2 -> 4
- net /A0-DAC: track 27.2 -> 27.6 mm, vias 1 -> 3
- net /SAM-~{RESET}: track 102.1 -> 102.3 mm, vias 7 -> 6
- added copper zone on F.Cu, net +4V
Other:
- rule pad_to_mask_clearance: 0.05 -> 0
- board text added: "3V SEL"

Commit message: Add files via upload
Parts:
- C13: value 0.01uF -> 10nF
- C20, C24, C26: value 47u -> 47uF
- moved C26 1.32 mm to (134.9, 111.6)
- moved G*** 1.21 mm to (101.6, 101.5)
- turned C20 to -90 degrees
Connections:
- C20 pad 1: GND -> +12V
- C20 pad 2: +12V -> GND
Routing:
- net GND: track 160.4 -> 246.5 mm, vias 138 -> 160
- net +4V: track 132.5 -> 131.2 mm
- net Net-(Q3-Pad1): track 4.97 -> 4.11 mm
Other:
- board text added: "0.0.2"
- board text removed: "Limited edition"

Commit message: Add files via upload
Parts:
- R22: value 52K3 -> 10K
Changed lines of the file:
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@@
       (effects (font (size 1 1) (thickness 0.15)))
     )
-    (fp_text value "52K3" (at 0 1.43) (layer "F.Fab")
+    (fp_text value "10K" (at 0 1.43) (layer "F.Fab")
       (effects (font (size 1 1) (thickness 0.15)))
     )

Commit message: Add files via upload
Routing:
- net Net-(D6-Pad2): track 13.3 -> 0.00 mm
- net GND: vias 160 -> 159
Changed lines of the file:
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@@
     (fp_line (start 6.1 4.5) (end 6.1 2.6) (layer "F.SilkS") (width 0.2))
     (fp_line (start 6.1 -4.5) (end -7.5 -4.5) (layer "F.SilkS") (width 0.2))
-    (fp_line (start -7.9 0) (end -7.9 0) (layer "F.SilkS") (width 0.1))
     (fp_line (start -7.5 4.5) (end 0.7 4.5) (layer "F.SilkS") (width 0.2))
     (fp_arc (start -8 0) (mid -7.95 -0.05) (end -7.9 0) (layer "F.SilkS") (width 0.1))
     (fp_arc (start -7.9 0) (mid -7.95 0.05) (end -8 0) (layer "F.SilkS") (width 0.1))
-    (fp_line (start -8.5 -5.5) (end 9.525 -5.5) (layer "F.CrtYd") (width 0.1))
-    (fp_line (start 9.525 7.925) (end -8.5 7.925) (layer "F.CrtYd") (width 0.1))
-    (fp_line (start -8.5 7.925) (end -8.5 -5.5) (layer "F.CrtYd") (width 0.1))
-    (fp_line (start 9.525 -5.5) (end 9.525 7.925) (layer "F.CrtYd") (width 0.1))
     (fp_line (start 6.1 4.5) (end 6.1 -4.5) (layer "F.Fab") (width 0.1))
     (fp_line (start -7.5 -4.5) (end -7.5 4.5) (layer "F.Fab") (width 0.1))
     (fp_line (start 6.1 -4.5) (end -7.5 -4.5) (layer "F.Fab") (width 0.1))
     (fp_line (start -7.5 4.5) (end 6.1 4.5) (layer "F.Fab") (width 0.1))
-    (pad "" np_thru_hole circle locked (at -1 3.5) (size 1.5 1.5) (drill 1.5) (layers *.Cu *.Mask))
-    (pad "" np_thru_hole circle locked (at -1 -3.5) (size 1.5 1.5) (drill 1.5) (layers *.Cu *.Mask))
-    (pad "1" thru_hole circle locked (at 0 0) (size 4.65 4.65) (drill 3.1) (layers *.Cu *.Mask)
+    (pad "" np_thru_hole circle (at -1 3.5) (size 1.5 1.5) (drill 1.5) (layers *.Cu *.Mask))
+    (pad "" np_thru_hole circle (at -1 -3.5) (size 1.5 1.5) (drill 1.5) (layers *.Cu *.Mask))
+    (pad "1" thru_hole circle (at 6.2 0) (size 4.65 4.65) (drill oval 1 3.1) (layers *.Cu *.Mask)
       (net 59 "Net-(D6-Pad2)") (pintype "passive"))
-    (pad "2" thru_hole circle locked (at 3.3 4.6) (size 4.65 4.65) (drill 3.1) (layers *.Cu *.Mask)
+    (pad "2" thru_hole circle (at 0 0) (size 4.65 4.65) (drill oval 1 3.1) (layers *.Cu *.Mask)
       (net 1 "GND") (pintype "passive"))
-    (pad "3" thru_hole circle locked (at 6.2 0) (size 4.65 4.65) (drill 3.1) (layers *.Cu *.Mask)
+    (pad "3" thru_hole circle (at 3.3 4.6) (size 4.65 4.65) (drill oval 3.1 1) (layers *.Cu *.Mask)
       (net 1 "GND") (pintype "passive"))
     (model "DC-005G-2.5A-2.0.stp"
@@
   (via (at 85.954 86.207) (size 0.5) (drill 0.25) (layers "F.Cu" "B.Cu") (free) (net 1))
   (via (at 139.182 98.975) (size 0.5) (drill 0.25) (layers "F.Cu" "B.Cu") (free) (net 1))
-  (via (at 94.734 115.169) (size 0.5) (drill 0.25) (layers "F.Cu" "B.Cu") (free) (net 1))
   (via (at 125.899 92) (size 0.5) (drill 0.25) (layers "F.Cu" "B.Cu") (net 1))
   (via (at 136.634 78.514) (size 0.5) (drill 0.25) (layers "F.Cu" "B.Cu") (free) (net 1))
@@
   (segment (start 92.796 97.783) (end 92.776 97.763) (width 0.225) (layer "B.Cu") (net 58))
   (segment (start 109.806 92.203) (end 109.806 92.344567) (width 0.225) (layer "B.Cu") (net 58))
-  (segment (start 89.216 113.138) (end 97.291 113.138) (width 0.6096) (layer "F.Cu") (net 59))
-  (segment (start 85.491 116.863) (end 89.216 113.138) (width 0.6096) (layer "F.Cu") (net 59))
   (segment (start 96.441 88.988) (end 95.851 88.988) (width 0.127) (layer "F.Cu") (net 64))
   (segment (start 95.407126 89.4695) (end 90.5005 89.4695) (width 0.127) (layer "F.Cu") (net 64))
@@
     )
   )
-  (zone (net 59) (net_name "Net-(D6-Pad2)") (layer "F.Cu") (hatch edge 0.508)
-    (priority 4)
-    (connect_pads yes (clearance 0.254))
-    (min_thickness 0.254) (filled_areas_thickness no)
-    (fill yes (thermal_gap 0.508) (thermal_bridge_width 0.508))
-    (polygon
-      (pts
-        (xy 98.466 114.603)
-        (xy 88.726 114.603)
-        (xy 88.726 118.033)
-        (xy 84.826 118.033)
-        (xy 84.826 112.113)
-        (xy 98.456 112.113)
-      )
-    )
-  )
   (zone (net 80) (net_name "+4V") (layer "F.Cu") (hatch edge 0.508)
     (priority 1)
@@
       )
     )
+  )
+  (zone (net 59) (net_name "Net-(D6-Pad2)") (layer "F.Cu") (hatch edge 0.508)
+    (priority 5)
+    (connect_pads yes (clearance 0.15))
+    (min_thickness 0.15) (filled_areas_thickness no)
+    (fill yes (thermal_gap 0.508) (thermal_bridge_width 0.508))
+    (polygon
+      (pts
+        (xy 98.5012 119.2276)
+        (xy 92.6592 119.2276)
+        (xy 91.5416 119.1768)
+        (xy 89.4588 117.2972)
+        (xy 89.0016 116.6368)
+        (xy 89.0016 112.1156)
+        (xy 98.5012 112.1156)
+      )
+    )
